Commit message: added kr6r900sixx inertia

File: kuka_kr6_support/urdf/kr6r900sixx_macro.xacro (robot description, xacro)
@@ -16,4 +16,12 @@
         </geometry>
       </collision>
+      <inertial>
+          <origin xyz="0 0 0" rpy="0 0 0" />
+          <mass value="0.1" />
+          <inertia
+            ixx="1.0" ixy="0.0" ixz="0.0"
+                      iyy="1.0" iyz="0.0"
+                                izz="1.0" />
+      </inertial>
     </link>
     <link name="${prefix}link_1">
@@ -30,4 +38,12 @@
         </geometry>
       </collision>
+      <inertial>
+          <origin xyz="0 0 0" rpy="0 0 0" />
+          <mass value="0.1" />
+          <inertia
+            ixx="1.0" ixy="0.0" ixz="0.0"
+                      iyy="1.0" iyz="0.0"
+                                izz="1.0" />
+      </inertial>
     </link>
     <link name="${prefix}link_2">
@@ -44,4 +60,12 @@
         </geometry>
       </collision>
+      <inertial>
+          <origin xyz="0 0 0" rpy="0 0 0" />
+          <mass value="0.1" />
+          <inertia
+            ixx="1.0" ixy="0.0" ixz="0.0"
+                      iyy="1.0" iyz="0.0"
+                                izz="1.0" />
+      </inertial>
     </link>
     <link name="${prefix}link_3">
@@ -58,4 +82,12 @@
         </geometry>
       </collision>
+      <inertial>
+          <origin xyz="0 0 0" rpy="0 0 0" />
+          <mass value="0.1" />
+          <inertia
+            ixx="1.0" ixy="0.0" ixz="0.0"
+                      iyy="1.0" iyz="0.0"
+                                izz="1.0" />
+      </inertial>
     </link>
     <link name="${prefix}link_4">
@@ -72,4 +104,12 @@
         </geometry>
       </collision>
+      <inertial>
+          <origin xyz="0 0 0" rpy="0 0 0" />
+          <mass value="0.1" />
+          <inertia
+            ixx="1.0" ixy="0.0" ixz="0.0"
+                      iyy="1.0" iyz="0.0"
+                                izz="1.0" />
+      </inertial>
     </link>
     <link name="${prefix}link_5">
@@ -86,4 +126,12 @@
         </geometry>
       </collision>
+      <inertial>
+          <origin xyz="0 0 0" rpy="0 0 0" />
+          <mass value="0.1" />
+          <inertia
+            ixx="1.0" ixy="0.0" ixz="0.0"
+                      iyy="1.0" iyz="0.0"
+                                izz="1.0" />
+      </inertial>
     </link>
     <link name="${prefix}link_6">
@@ -100,4 +148,12 @@
         </geometry>
       </collision>
+      <inertial>
+          <origin xyz="0 0 0" rpy="0 0 0" />
+          <mass value="0.1" />
+          <inertia
+            ixx="1.0" ixy="0.0" ixz="0.0"
+                      iyy="1.0" iyz="0.0"
+                                izz="1.0" />
+      </inertial>
     </link>
     <!-- This frame corresponds to the $FLANGE coordinate system in KUKA KRC controllers. -->
@@ -109,4 +165,5 @@
       <axis xyz="0 0 -1"/>
       <limit effort="0" lower="${-DEG2RAD * 170}" upper="${DEG2RAD * 170}" velocity="${DEG2RAD * 360}"/>
+      <dynamics damping="100.0" friction="100.0"/>
     </joint>
     <joint name="${prefix}joint_a2" type="revolute">
@@ -116,4 +173,5 @@
       <axis xyz="0 1 0"/>
       <limit effort="0" lower="${-DEG2RAD * 190}" upper="${DEG2RAD * 45}" velocity="${DEG2RAD * 300}"/>
+      <dynamics damping="100.0" friction="100.0"/>
     </joint>
     <joint name="${prefix}joint_a3" type="revolute">
@@ -123,4 +181,5 @@
       <axis xyz="0 1 0"/>
       <limit effort="0" lower="${-DEG2RAD * 120}" upper="${DEG2RAD * 156}" velocity="${DEG2RAD * 360}"/>
+      <dynamics damping="100.0" friction="100.0"/>
     </joint>
     <joint name="${prefix}joint_a4" type="revolute">
@@ -130,4 +189,5 @@
       <axis xyz="-1 0 0"/>
       <limit effort="0" lower="${-DEG2RAD * 185}" upper="${DEG2RAD * 185}" velocity="${DEG2RAD * 381}"/>
+      <dynamics damping="100.0" friction="100.0"/>
     </joint>
     <joint name="${prefix}joint_a5" type="revolute">
@@ -137,4 +197,5 @@
       <axis xyz="0 1 0"/>
       <limit effort="0" lower="${-DEG2RAD * 120}" upper="${DEG2RAD * 120}" velocity="${DEG2RAD * 388}"/>
+      <dynamics damping="100.0" friction="100.0"/>
     </joint>
     <joint name="${prefix}joint_a6" type="revolute">
@@ -144,4 +205,5 @@
       <axis xyz="-1 0 0"/>
       <limit effort="0" lower="${-DEG2RAD * 350}" upper="${DEG2RAD * 350}" velocity="${DEG2RAD * 615}"/>
+      <dynamics damping="100.0" friction="100.0"/>
     </joint>
     <joint name="${prefix}joint_a6-tool0" type="fixed">
@@ -157,4 +219,58 @@
       <child link="${prefix}base"/>
     </joint>
+    <transmission name="${prefix}joint_a1_trans">
+      <type>transmission_interface/SimpleTransmission</type>
+      <joint name="${prefix}joint_a1">
+        <hardwareInterface>PositionJointInterface</hardwareInterface>
+      </joint>
+      <actuator name="${prefix}joint_a1_motor">
+        <mechanicalReduction>1</mechanicalReduction>
+      </actuator>
+    </transmission>
+    <transmission name="${prefix}joint_a2_trans">
+      <type>transmission_interface/SimpleTransmission</type>
+      <joint name="${prefix}joint_a2">
+        <hardwareInterface>PositionJointInterface</hardwareInterface>
+      </joint>
+      <actuator name="${prefix}joint_a2_motor">
+        <mechanicalReduction>1</mechanicalReduction>
+      </actuator>
+    </transmission>
+    <transmission name="${prefix}joint_a3_trans">
+      <type>transmission_interface/SimpleTransmission</type>
+      <joint name="${prefix}joint_a3">
+        <hardwareInterface>PositionJointInterface</hardwareInterface>
+      </joint>
+      <actuator name="${prefix}joint_a3_motor">
+        <mechanicalReduction>1</mechanicalReduction>
+      </actuator>
+    </transmission>
+    <transmission name="${prefix}joint_a4_trans">
+      <type>transmission_interface/SimpleTransmission</type>
+      <joint name="${prefix}joint_a4">
+        <hardwareInterface>PositionJointInterface</hardwareInterface>
+      </joint>
+      <actuator name="${prefix}joint_a4_motor">
+        <mechanicalReduction>1</mechanicalReduction>
+      </actuator>
+    </transmission>
+    <transmission name="${prefix}joint_a5_trans">
+      <type>transmission_interface/SimpleTransmission</type>
+      <joint name="${prefix}joint_a5">
+        <hardwareInterface>PositionJointInterface</hardwareInterface>
+      </joint>
+      <actuator name="${prefix}joint_a5_motor">
+        <mechanicalReduction>1</mechanicalReduction>
+      </actuator>
+    </transmission>
+    <transmission name="${prefix}joint_a6_trans">
+      <type>transmission_interface/SimpleTransmission</type>
+      <joint name="${prefix}joint_a6">
+        <hardwareInterface>PositionJointInterface</hardwareInterface>
+      </joint>
+      <actuator name="${prefix}joint_a6_motor">
+        <mechanicalReduction>1</mechanicalReduction>
+      </actuator>
+    </transmission>
   </xacro:macro>
 </robot>
