Commit message: first migration commit

File: kuka_kr10_support/urdf/kr10r1100sixx_macro.xacro (robot description, xacro)
@@ -8,5 +8,5 @@
         <origin xyz="0 0 0" rpy="0 0 0"/>
         <geometry>
-          <mesh filename="package://kuka_kr10_support/meshes/kr10r1100sixx/visual/base_link.stl" />
+          <mesh filename="package://kuka_kr10_support/meshes/kr10r1100sixx/visual/base.stl" />
         </geometry>
         <xacro:material_kuka_black />
@@ -15,5 +15,5 @@
         <origin xyz="0 0 0" rpy="0 0 0"/>
         <geometry>
-          <mesh filename="package://kuka_kr10_support/meshes/kr10r1100sixx/collision/base_link.stl" />
+          <mesh filename="package://kuka_kr10_support/meshes/kr10r1100sixx/collision/base.stl" />
         </geometry>
       </collision>
@@ -109,6 +109,6 @@
       </collision>
     </link>
-    <!-- Following REP199, this frame shall be use to attach EEF or other equipment -->
-    <link name="${prefix}flange" />
+    <!-- This frame corresponds to the $FLANGE coordinate system in KUKA KRC controllers. -->
+    <link name="${prefix}tool0"/>
     <joint name="${prefix}joint_a1" type="revolute">
       <origin xyz="0 0 0.400" rpy="0 0 0"/>
@@ -116,5 +116,5 @@
       <child link="${prefix}link_1"/>
       <axis xyz="0 0 -1"/>
-      <limit effort="0" lower="${radians(-170)}" upper="${radians(170)}" velocity="${radians(300)}"/>
+      <limit effort="0" lower="${-DEG2RAD * 170}" upper="${DEG2RAD * 170}" velocity="${DEG2RAD * 360}"/>
     </joint>
     <joint name="${prefix}joint_a2" type="revolute">
@@ -123,5 +123,5 @@
       <child link="${prefix}link_2"/>
       <axis xyz="0 1 0"/>
-      <limit effort="0" lower="${radians(-190)}" upper="${radians(45)}" velocity="${radians(225)}"/>
+      <limit effort="0" lower="${-DEG2RAD * 190}" upper="${DEG2RAD * 45}" velocity="${DEG2RAD * 300}"/>
     </joint>
     <joint name="${prefix}joint_a3" type="revolute">
@@ -130,5 +130,5 @@
       <child link="${prefix}link_3"/>
       <axis xyz="0 1 0"/>
-      <limit effort="0" lower="${radians(-120)}" upper="${radians(156)}" velocity="${radians(225)}"/>
+      <limit effort="0" lower="${-DEG2RAD * 120}" upper="${DEG2RAD * 156}" velocity="${DEG2RAD * 360}"/>
     </joint>
     <joint name="${prefix}joint_a4" type="revolute">
@@ -137,5 +137,5 @@
       <child link="${prefix}link_4"/>
       <axis xyz="-1 0 0"/>
-      <limit effort="0" lower="${radians(-185)}" upper="${radians(185)}" velocity="${radians(381)}"/>
+      <limit effort="0" lower="${-DEG2RAD * 185}" upper="${DEG2RAD * 185}" velocity="${DEG2RAD * 381}"/>
     </joint>
     <joint name="${prefix}joint_a5" type="revolute">
@@ -144,5 +144,5 @@
       <child link="${prefix}link_5"/>
       <axis xyz="0 1 0"/>
-      <limit effort="0" lower="${radians(-120)}" upper="${radians(120)}" velocity="${radians(311)}"/>
+      <limit effort="0" lower="${-DEG2RAD * 120}" upper="${DEG2RAD * 120}" velocity="${DEG2RAD * 388}"/>
     </joint>
     <joint name="${prefix}joint_a6" type="revolute">
@@ -151,10 +151,10 @@
       <child link="${prefix}link_6"/>
       <axis xyz="-1 0 0"/>
-      <limit effort="0" lower="${radians(-350)}" upper="${radians(350)}" velocity="${radians(492)}"/>
+      <limit effort="0" lower="${-DEG2RAD * 350}" upper="${DEG2RAD * 350}" velocity="${DEG2RAD * 615}"/>
     </joint>
-    <joint name="${prefix}joint_a6-flange" type="fixed">
+    <joint name="${prefix}joint_a6-tool0" type="fixed">
       <parent link="${prefix}link_6"/>
-      <child link="${prefix}flange"/>
-      <origin xyz="0 0 0" rpy="0 0 0"/>
+      <child link="${prefix}tool0"/>
+      <origin xyz="0 0 0" rpy="0 ${DEG2RAD * 90} 0"/>
     </joint>
     <!-- ROS base_link to KUKA $ROBROOT coordinate system transform -->
@@ -165,11 +165,4 @@
       <child link="${prefix}base"/>
     </joint>
-    <!-- This frame corresponds to the $TOOL coordinate system in KUKA KRC controllers -->
-    <link name="${prefix}tool0" />
-    <joint name="${prefix}flange-tool0" type="fixed">
-      <parent link="${prefix}flange"/>
-      <child link="${prefix}tool0"/>
-      <origin xyz="0 0 0" rpy="0 ${radians(90)} 0"/>
-    </joint>
   </xacro:macro>
 </robot>

File: kuka_resources/urdf/common_colours.xacro (robot description, xacro)
@@ -72,9 +72,3 @@
   <!-- RAL 9002 - gray white  -->
   <xacro:property name="colour_kuka_ral_gray_white"       value="${215/255} ${213/255} ${203/255} 1.0" />
-  <!-- RAL 9007 - grey aluminium -->
-  <xacro:property name="colour_kuka_ral_gray_aluminium"   value="${135/255} ${133/255} ${129/255} 1.0" />
-  <!-- RAL 9010 - pure white  -->
-  <xacro:property name="colour_kuka_ral_pure_white"       value="${241/255} ${236/255} ${255/255} 1.0" />
-  <!-- RAL 9016 - traffic white -->
-  <xacro:property name="colour_kuka_ral_traffic_white"    value="${241/255}  ${240/255} ${234/255} 1.0" />
 </robot>

File: kuka_resources/urdf/common_materials.xacro (robot description, xacro)
@@ -152,18 +152,3 @@
     </material>
   </xacro:macro>
-  <xacro:macro name="material_kuka_ral_gray_aluminium">
-    <material name="">
-      <color rgba="${colour_kuka_ral_gray_aluminium}"/>
-    </material>
-  </xacro:macro>
-  <xacro:macro name="material_kuka_ral_pure_white">
-    <material name="">
-      <color rgba="${colour_kuka_ral_pure_white}"/>
-    </material>
-  </xacro:macro>
-  <xacro:macro name="material_kuka_ral_traffic_white">
-    <material name="">
-      <color rgba="${colour_kuka_ral_traffic_white}"/>
-    </material>
-  </xacro:macro>
 </robot>
